File: heatplat.kicad_pcb (KiCad board)
At the start: 2 copper layers, 99.1 x 99.1 mm, 14 parts, among them J1 Barrel_Jack_Switch

Commit message: update resister values
Parts:
- R5, R6: value R -> 2R2
Changed lines of the file:
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@@
-(kicad_pcb (version 20171130) (host pcbnew 5.1.2-f72e74a~84~ubuntu18.04.1)
+(kicad_pcb (version 20171130) (host pcbnew "(5.1.2)-2")
   (general
     (thickness 1.6)
@@
   )
   (setup
-    (last_trace_width 5.08)
+    (last_trace_width 0.25)
     (user_trace_width 0.2032)
     (user_trace_width 1.27)
@@
     (aux_axis_origin 0 0)
     (grid_origin 77.47 -76.2)
-    (visible_elements FFFFFF7F)
+    (visible_elements 7FFFFFFF)
     (pcbplotparams
       (layerselection 0x010fc_ffffffff)
@@
       (effects (font (size 1 1) (thickness 0.15)))
     )
-    (fp_text value R (at 35.56 0) (layer F.Fab)
+    (fp_text value 2R2 (at 35.56 0) (layer F.Fab)
       (effects (font (size 1 1) (thickness 0.15)))
     )
@@
       (effects (font (size 1 1) (thickness 0.15)))
     )
-    (fp_text value R (at 20.32 0) (layer F.Fab)
-      (effects (font (size 1 1) (thickness 0.15)))
-    )
+    (fp_text value 2R2 (at 20.32 0) (layer F.Fab)
+      (effects (font (size 1 1) (thickness 0.15)))
+    )
